File: EagleSkatch/ArduinoNanoA6cConnectorBoard/board.brd (EAGLE design)
At the start: 79.7 x 61 mm, 14 parts, among them J1 POWER_JACKSLT

Commit message: Boarddesign finnished
Finished Board design and send it to seed studio
Connections:
- removed net N$3: IN-.1, J1.GND@1, J1.GND@2, J2.GND1
- new net N$12: A6CL.4, NANO3R.5
- new net N$13: A6CL.5, NANO3R.6
- net GND: now also IN-.1, J1.GND@1, J1.GND@2, J2.GND1
Routing:
- net N$3: track 25.7 -> 0.00 mm
- net GND: track 0.00 -> 14.3 mm
- net VCC: track 102.5 -> 111.1 mm
- net N$10: track 38.0 -> 29.9 mm
- net N$9: track 7.18 -> 0.00 mm, vias 1 -> 0
- net N$11: track 6.38 -> 0.00 mm, vias 1 -> 0
- net N$13: track 0.00 -> 6.05 mm
- net N$12: track 0.00 -> 6.05 mm
- net N$1: track 32.2 -> 27.8 mm
Other:
- board text added: "JS"
Changed lines of the file:
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@@
 <hole x="12.7" y="17.78" drill="1"/>
 <hole x="58.42" y="17.78" drill="1"/>
+<text x="64.77" y="7.62" size="1.778" layer="16" rot="MR0">JS</text>
 </plain>
 <attributes>
@@
 <contactref element="A6CL" pad="11"/>
 <wire x1="35.306" y1="51.773" x2="35.306" y2="56.896" width="0.4064" layer="16"/>
-<wire x1="36.83" y1="58.42" x2="50.8" y2="58.42" width="0.4064" layer="16"/>
-<wire x1="50.8" y1="58.42" x2="52.07" y2="57.15" width="0.4064" layer="16"/>
+<wire x1="36.83" y1="58.42" x2="43.18" y2="58.42" width="0.4064" layer="16"/>
+<wire x1="43.18" y1="58.42" x2="44.958" y2="56.007" width="0.4064" layer="16"/>
 <wire x1="35.306" y1="56.896" x2="36.83" y2="58.42" width="0.4064" layer="16"/>
-<via x="52.07" y="57.15" extent="1-16" drill="0.35"/>
-<wire x1="52.07" y1="57.15" x2="52.07" y2="46.99" width="0.4064" layer="1"/>
-<via x="52.07" y="46.99" extent="1-16" drill="0.35"/>
-<wire x1="52.07" y1="46.99" x2="50.8" y2="45.72" width="0.4064" layer="16"/>
-<wire x1="50.8" y1="45.72" x2="47.921" y2="45.72" width="0.4064" layer="16"/>
+<via x="44.958" y="56.007" extent="1-16" drill="0.35"/>
+<wire x1="44.958" y1="56.007" x2="44.958" y2="45.847" width="0.4064" layer="1"/>
+<via x="44.958" y="45.847" extent="1-16" drill="0.35"/>
+<wire x1="44.958" y1="45.847" x2="47.879" y2="45.72" width="0.4064" layer="16"/>
+<wire x1="47.879" y1="45.72" x2="47.921" y2="45.72" width="0.4064" layer="16"/>
 <wire x1="47.921" y1="45.72" x2="47.844" y2="45.797" width="0.4064" layer="16"/>
 </signal>
@@
 <contactref element="OUT-" pad="1"/>
 <contactref element="NANO3L" pad="2"/>
-<polygon width="0.4064" layer="16">
-<vertex x="-5.08" y="66.04"/>
-<vertex x="88.9" y="66.04"/>
-<vertex x="88.9" y="-20.32"/>
-<vertex x="-10.16" y="-19.05"/>
-<vertex x="-7.62" y="5.08"/>
-<vertex x="3.81" y="3.81"/>
-<vertex x="10.16" y="3.81"/>
-<vertex x="13.97" y="7.62"/>
-<vertex x="24.13" y="7.62"/>
-<vertex x="24.13" y="17.78"/>
-<vertex x="19.05" y="19.05"/>
-<vertex x="13.97" y="13.97"/>
-<vertex x="8.89" y="13.97"/>
-<vertex x="6.35" y="17.78"/>
-<vertex x="5.08" y="19.05"/>
-<vertex x="-5.08" y="19.05"/>
+<contactref element="IN-" pad="1"/>
+<contactref element="J2" pad="GND1"/>
+<contactref element="J1" pad="GND@2"/>
+<contactref element="J1" pad="GND@1"/>
+<polygon width="0.508" layer="16">
+<vertex x="-20.32" y="19.05"/>
+<vertex x="-21.59" y="-13.97"/>
+<vertex x="109.22" y="-11.43"/>
+<vertex x="81.28" y="87.63"/>
+<vertex x="-29.21" y="80.01"/>
+<vertex x="-20.32" y="22.86"/>
 </polygon>
-<polygon width="0.4064" layer="16">
-<vertex x="-5.08" y="66.04"/>
-<vertex x="102.87" y="69.85"/>
-<vertex x="92.71" y="-19.05"/>
-<vertex x="-17.78" y="-22.86"/>
+<polygon width="0.508" layer="1">
+<vertex x="-41.91" y="59.69"/>
+<vertex x="-36.83" y="-33.02"/>
+<vertex x="149.86" y="-35.56"/>
+<vertex x="87.63" y="130.81"/>
+<vertex x="-44.45" y="114.3"/>
 </polygon>
-<polygon width="0.4064" layer="1">
-<vertex x="-15.24" y="-7.62"/>
-<vertex x="96.52" y="-7.62"/>
-<vertex x="90.17" y="68.58"/>
-<vertex x="-20.32" y="62.23"/>
-<vertex x="-15.24" y="39.37"/>
-</polygon>
+<wire x1="22.89" y1="3.97" x2="22.89" y2="6.35" width="0.4064" layer="1"/>
+<wire x1="22.89" y1="6.35" x2="22.86" y2="6.35" width="0.4064" layer="1"/>
+<wire x1="22.86" y1="6.35" x2="22.86" y2="16.51" width="0.4064" layer="1"/>
+<wire x1="22.86" y1="16.51" x2="21.11" y2="16.51" width="0.4064" layer="1"/>
 </signal>
 <signal name="VCC">
@@
 <wire x1="3.81" y1="35.56" x2="20.32" y2="20.32" width="0.4064" layer="16"/>
 <wire x1="26.67" y1="19.05" x2="30.48" y2="15.24" width="0.4064" layer="16"/>
-<wire x1="30.48" y1="15.24" x2="43.18" y2="15.24" width="0.4064" layer="16"/>
-<wire x1="43.18" y1="15.24" x2="44.45" y2="16.51" width="0.4064" layer="16"/>
-<wire x1="44.45" y1="16.51" x2="44.45" y2="44.943" width="0.4064" layer="16"/>
-<wire x1="44.45" y1="44.943" x2="47.844" y2="48.337" width="0.4064" layer="16"/>
-</signal>
-<signal name="N$1">
-<contactref element="IN+" pad="1"/>
-<contactref element="J2" pad="VBUS1"/>
-<contactref element="J1" pad="PWR"/>
-<wire x1="20.29" y1="3.97" x2="20.29" y2="5.11" width="0.4064" layer="1"/>
-<wire x1="20.29" y1="5.11" x2="19.05" y2="6.35" width="0.4064" layer="1"/>
-<wire x1="19.05" y1="6.35" x2="13.97" y2="6.35" width="0.4064" layer="1"/>
-<wire x1="10.16" y1="2.54" x2="1.27" y2="2.54" width="0.4064" layer="1"/>
-<wire x1="1.27" y1="2.54" x2="1.27" y2="7.41" width="0.4064" layer="1"/>
-<wire x1="13.97" y1="6.35" x2="10.16" y2="2.54" width="0.4064" layer="1"/>
-<wire x1="6.39" y1="12.53" x2="6.39" y2="13.93" width="0.6096" layer="16"/>
-<wire x1="6.39" y1="13.93" x2="3.81" y2="16.51" width="0.6096" layer="16"/>
-<wire x1="1.27" y1="7.41" x2="6.39" y2="12.53" width="0" layer="19" extent="1-1"/>
-</signal>
-<signal name="N$3">
-<contactref element="J1" pad="GND@1"/>
-<contactref element="J1" pad="GND@2"/>
-<contactref element="J2" pad="GND1"/>
-<contactref element="IN-" pad="1"/>
-<wire x1="6.39" y1="6.23" x2="8.09" y2="6.23" width="0.508" layer="16"/>
-<wire x1="8.09" y1="6.23" x2="11.39" y2="9.53" width="0.508" layer="16"/>
-<wire x1="11.39" y1="9.53" x2="14.13" y2="9.53" width="0.508" layer="16"/>
-<wire x1="14.13" y1="9.53" x2="21.11" y2="16.51" width="0.508" layer="16"/>
-<wire x1="22.89" y1="3.97" x2="22.89" y2="8.86" width="0.4064" layer="1"/>
-<wire x1="22.89" y1="8.86" x2="21.59" y2="10.16" width="0.4064" layer="1"/>
-<wire x1="21.11" y1="16.51" x2="21.59" y2="10.16" width="0" layer="19" extent="1-1"/>
+<wire x1="30.48" y1="15.24" x2="49.53" y2="15.24" width="0.4064" layer="16"/>
+<wire x1="53.34" y1="19.05" x2="53.34" y2="43.673" width="0.4064" layer="16"/>
+<wire x1="53.34" y1="43.673" x2="47.844" y2="48.337" width="0.4064" layer="16"/>
+<wire x1="49.53" y1="15.24" x2="53.34" y2="19.05" width="0.4064" layer="16"/>
 </signal>
 <signal name="N$2">
@@
 <wire x1="67.31" y1="22.86" x2="73.66" y2="22.86" width="0.508" layer="16"/>
 </signal>
-<signal name="N$9">
-<via x="1.27" y="7.62" extent="1-16" drill="0.35"/>
-<wire x1="1.27" y1="7.62" x2="6.35" y2="12.7" width="0.6096" layer="16"/>
-</signal>
-<signal name="N$11">
-<via x="21.59" y="10.16" extent="1-16" drill="0.35"/>
-<wire x1="21.59" y1="10.16" x2="21.59" y2="16.002" width="0.6096" layer="16"/>
-<wire x1="21.59" y1="16.002" x2="21.209" y2="16.383" width="0.6096" layer="16"/>
+<signal name="N$12">
+<contactref element="NANO3R" pad="5"/>
+<contactref element="A6CL" pad="4"/>
+<wire x1="41.91" y1="29.21" x2="47.844" y2="28.017" width="0.508" layer="16"/>
+</signal>
+<signal name="N$13">
+<contactref element="NANO3R" pad="6"/>
+<contactref element="A6CL" pad="5"/>
+<wire x1="41.91" y1="31.75" x2="47.844" y2="30.557" width="0.508" layer="16"/>
+</signal>
+<signal name="N$1">
+<contactref element="J2" pad="VBUS1"/>
+<contactref element="IN+" pad="1"/>
+<contactref element="J1" pad="PWR"/>
+<wire x1="20.29" y1="3.97" x2="20.29" y2="11.46" width="0.4064" layer="1"/>
+<wire x1="20.29" y1="11.46" x2="17.78" y2="13.97" width="0.4064" layer="1"/>
+<wire x1="17.78" y1="13.97" x2="7.83" y2="13.97" width="0.4064" layer="1"/>
+<wire x1="7.83" y1="13.97" x2="6.39" y2="12.53" width="0.4064" layer="1"/>
+<wire x1="6.39" y1="12.53" x2="3.81" y2="16.51" width="0.508" layer="16"/>
 </signal>
 </signals>
